File: pcbs/iuhr.brd (EAGLE design)
At the start: 38.4 x 23 mm, 84 parts, among them Q1 20.000MHz, Q2 MOSFET-NCHANNELSMD

Commit message: Separate logic and power ground.
Routing:
- net GND: track 155.2 -> 153.4 mm, vias 42 -> 41
Changed lines of the file:
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@@
 <layer number="14" name="Route14" color="1" fill="6" visible="no" active="no"/>
 <layer number="15" name="Route15" color="4" fill="6" visible="no" active="no"/>
-<layer number="16" name="Bottom" color="1" fill="1" visible="no" active="yes"/>
+<layer number="16" name="Bottom" color="1" fill="1" visible="yes" active="yes"/>
 <layer number="17" name="Pads" color="2" fill="1" visible="yes" active="yes"/>
 <layer number="18" name="Vias" color="2" fill="1" visible="yes" active="yes"/>
@@
 <layer number="20" name="Dimension" color="15" fill="1" visible="yes" active="yes"/>
 <layer number="21" name="tPlace" color="7" fill="1" visible="yes" active="yes"/>
-<layer number="22" name="bPlace" color="7" fill="1" visible="no" active="yes"/>
+<layer number="22" name="bPlace" color="7" fill="1" visible="yes" active="yes"/>
 <layer number="23" name="tOrigins" color="15" fill="1" visible="yes" active="yes"/>
-<layer number="24" name="bOrigins" color="15" fill="1" visible="no" active="yes"/>
-<layer number="25" name="tNames" color="7" fill="1" visible="yes" active="yes"/>
+<layer number="24" name="bOrigins" color="15" fill="1" visible="yes" active="yes"/>
+<layer number="25" name="tNames" color="7" fill="1" visible="no" active="yes"/>
 <layer number="26" name="bNames" color="7" fill="1" visible="no" active="yes"/>
 <layer number="27" name="tValues" color="7" fill="1" visible="no" active="yes"/>
@@
 <layer number="38" name="bTest" color="7" fill="1" visible="no" active="yes"/>
 <layer number="39" name="tKeepout" color="4" fill="11" visible="yes" active="yes"/>
-<layer number="40" name="bKeepout" color="1" fill="11" visible="no" active="yes"/>
+<layer number="40" name="bKeepout" color="1" fill="11" visible="yes" active="yes"/>
 <layer number="41" name="tRestrict" color="4" fill="10" visible="no" active="yes"/>
 <layer number="42" name="bRestrict" color="1" fill="10" visible="no" active="yes"/>
@@
 <wire x1="14.4" y1="7.6" x2="14.4" y2="7.65" width="0.3" layer="16"/>
 <wire x1="14.4" y1="7.65" x2="13.6" y2="8.65" width="0.3" layer="16"/>
-<wire x1="11.6" y1="7.8" x2="12.4" y2="8.6" width="0.5" layer="16"/>
-<wire x1="12.4" y1="8.6" x2="12.6" y2="8.6" width="0.5" layer="16"/>
-<wire x1="12.6" y1="8.6" x2="13.35" y2="8.6" width="0.5" layer="16"/>
 <wire x1="13.35" y1="8.6" x2="13.6" y2="8.65" width="0.5" layer="16"/>
 <wire x1="11.6" y1="7.8" x2="10" y2="7.8" width="0.3" layer="16"/>
 <wire x1="10" y1="7.8" x2="8.2" y2="9.6" width="0.3" layer="16"/>
 <via x="8.2" y="9.6" extent="1-16" drill="0.3302"/>
-<wire x1="13.6" y1="5.65" x2="12.75" y2="5.65" width="0.5" layer="16"/>
-<wire x1="12.75" y1="5.65" x2="12.6" y2="5.8" width="0.5" layer="16"/>
-<wire x1="12.6" y1="5.8" x2="12.6" y2="8.6" width="0.5" layer="16"/>
 <polygon width="0.2" layer="1" isolate="0.3">
 <vertex x="0" y="23"/>
@@
 <via x="12.2" y="10.4" extent="1-16" drill="0.3302"/>
 <via x="13.8" y="10.4" extent="1-16" drill="0.3302"/>
-<via x="13" y="9.6" extent="1-16" drill="0.3302"/>
 <via x="9" y="8.8" extent="1-16" drill="0.3302"/>
 <via x="9.8" y="8" extent="1-16" drill="0.3302"/>
@@
 <wire x1="35" y1="8.2" x2="35" y2="7" width="0.5" layer="16"/>
 <wire x1="35" y1="7" x2="34.8" y2="6.8" width="0.5" layer="16"/>
-<polygon width="0.2" layer="16" isolate="0.3">
-<vertex x="0" y="23"/>
-<vertex x="38.4" y="23"/>
-<vertex x="38.4" y="0"/>
-<vertex x="0" y="0"/>
-</polygon>
 <wire x1="15.2" y1="17" x2="17" y2="17" width="1" layer="16"/>
 <wire x1="17" y1="17" x2="18.6" y2="18.6" width="1" layer="16"/>
@@
 <wire x1="5" y1="19.2" x2="5" y2="21.8" width="0.3" layer="16"/>
 <wire x1="5" y1="21.8" x2="6.6" y2="22.2" width="0.3" layer="16"/>
+<wire x1="13.6" y1="8.65" x2="13.25" y2="8.65" width="0.2" layer="16"/>
+<wire x1="13.25" y1="8.65" x2="12.8" y2="8.2" width="0.2" layer="16"/>
+<wire x1="12.8" y1="8.2" x2="12.8" y2="6" width="0.2" layer="16"/>
+<wire x1="12.8" y1="6" x2="13" y2="5.8" width="0.2" layer="16"/>
+<wire x1="13" y1="5.8" x2="13.45" y2="5.8" width="0.2" layer="16"/>
+<wire x1="13.45" y1="5.8" x2="13.6" y2="5.65" width="0.2" layer="16"/>
+<polygon width="0.2" layer="16" isolate="0.3">
+<vertex x="0" y="23"/>
+<vertex x="38.4" y="23"/>
+<vertex x="38.4" y="0"/>
+<vertex x="13" y="0"/>
+<vertex x="13" y="9.2"/>
+<vertex x="14.6" y="9.2"/>
+<vertex x="14.6" y="9.6"/>
+<vertex x="12.4" y="9.6"/>
+<vertex x="12.4" y="0"/>
+<vertex x="0" y="0"/>
+</polygon>
 </signal>
 <signal name="VCC">
